Commit message: v0.3 material

File: robot.urdf (robot description, URDF)
Before this commit: robot demo-robot-description, 5 links, 4 joints
Links:
- link base: mass 1e-09 -> 411.176
- link hip: mass 1e-09 -> 7.41924
- link pelvis_2: mass 1e-09 -> 14.426

Commit message: v0.4

File: robot.urdf (robot description, URDF)
Before this commit: robot demo-robot-description, 5 links, 4 joints
Links:
- link base: geometry collision mesh filename=package://assets/base.stl; visual mesh filename=package://assets/base.stl
- link hip: geometry collision mesh filename=package://assets/hip.stl; visual mesh filename=package://assets/hip.stl
- link pelvis_2: geometry collision mesh filename=package://assets/pelvis.stl; visual mesh filename=package://assets/pelvis.stl

Commit message: v0.5

File: robot.urdf (robot description, URDF)
Before this commit: robot demo-robot-description, 5 links, 4 joints
Links:
- removed link base
- removed link hip
- removed link pelvis_2
- added link l_hip_assembly, mass 7.41924; collision mesh filename=assets/hip.stl; visual mesh filename=assets/hip.stl
- added link pelvis_assembly, mass 14.426; collision mesh filename=assets/pelvis.stl; visual mesh filename=assets/pelvis.stl
- added link torso_assembly, mass 411.176; collision mesh filename=assets/base.stl; visual mesh filename=assets/base.stl
Joints:
- joint left_hip_frame: origin xyz=-1.53081e-19 0 -2.77556e-17 rpy=-1.5708 -1.5708 0 -> xyz=2.84603e-19 0 0 rpy=-1.5708 -1.5708 0; parent hip -> l_hip_assembly
- joint left_hip_pitch_joint: child hip -> l_hip_assembly; limit lower=-3.141592653589793 upper=3.141592653589793 effort=10 velocity=10 -> lower=-1.74533 upper=0.785398 effort=10 velocity=10; origin xyz=-0.12 1.99005e-18 -0.127 rpy=1.5708 -0 1.5708 -> xyz=-0.123 -3.35425e-18 -0.127 rpy=1.5708 -5.83786e-16 1.5708; parent pelvis_2 -> pelvis_assembly
- joint pelvis_frame: origin xyz=7.59908e-17 4.77612e-18 0 rpy=0 -0 0 -> xyz=2.71051e-17 -1.63816e-18 0 rpy=4.1926e-34 -1.08683e-34 5.79718e-19; parent pelvis_2 -> pelvis_assembly
- joint waist_yaw_joint: child pelvis_2 -> pelvis_assembly; limit lower=-3.141592653589793 upper=3.141592653589793 effort=10 velocity=10 -> lower=-0.809362 upper=0.761434 effort=10 velocity=10; origin xyz=-3.81639e-16 -1.99005e-18 0.732 rpy=0 -0 0 -> xyz=0.000624923 -1.11573e-17 -0.298822 rpy=-2.52536e-18 -4.61573e-19 0.0239641; parent base -> torso_assembly

Commit message: v0.6

File: robot.urdf (robot description, URDF)
Before this commit: robot demo-robot-description, 5 links, 4 joints
Links:
- removed link left_hip
- removed link pelvis
- removed link torso_assembly
- added link base, mass 356.291; collision mesh filename=assets/base.stl; visual mesh filename=assets/base.stl
- added link l_ankle_assembly, mass 1e-09; collision mesh filename=assets/frame.stl; collision mesh filename=assets/l_ankle.stl
- added link l_ankle_assembly_2, mass 1e-09; collision mesh filename=assets/frame.stl; collision mesh filename=assets/l_ankle.stl
- added link l_elbow_assembly, mass 1e-09; collision mesh filename=assets/frame.stl; collision mesh filename=assets/l_elbow.stl
- added link l_foot_assembly, mass 1e-09; collision mesh filename=assets/frame.stl; collision mesh filename=assets/l_foot.stl
- added link l_foot_assembly_2, mass 1e-09; collision mesh filename=assets/frame.stl; collision mesh filename=assets/l_foot.stl
- added link l_forearm_linkage_assembly, mass 1e-09; collision mesh filename=assets/frame.stl; collision mesh filename=assets/l_forearm_linkage.stl
- added link l_lower_femur_assembly, mass 1e-09; collision mesh filename=assets/frame.stl; collision mesh filename=assets/l_lower_femur.stl
- added link l_lower_forearm_assembly, mass 1e-09; collision mesh filename=assets/frame.stl; collision mesh filename=assets/l_lower_forearm.stl
- added link l_shoulder_assembly, mass 1e-09; collision mesh filename=assets/frame.stl; collision mesh filename=assets/l_shoulder.stl
- added link l_tibia_assembly, mass 1e-09; collision mesh filename=assets/frame.stl; collision mesh filename=assets/l_tibia.stl
- added link l_upper_arm_assembly, mass 1e-09; collision mesh filename=assets/frame.stl; collision mesh filename=assets/l_upper_arm.stl
- added link l_upper_femur_assembly, mass 1e-09; collision mesh filename=assets/frame.stl; collision mesh filename=assets/l_upper_femur.stl
- added link l_upper_forearm_assembly, mass 1e-09; collision mesh filename=assets/frame.stl; collision mesh filename=assets/l_upper_forearm.stl
- added link l_wrist_assembly, mass 1e-09; collision mesh filename=assets/frame.stl; collision mesh filename=assets/l_wrist.stl
- added link r_elbow_assembly, mass 1e-09; collision mesh filename=assets/frame.stl; collision mesh filename=assets/r_elbow.stl
- added link r_forearm_linkage_assembly, mass 1e-09; collision mesh filename=assets/frame.stl; collision mesh filename=assets/r_forearm_linkage.stl
- added link r_hip_assembly, mass 6.32737; collision mesh filename=assets/r_hip.stl; visual mesh filename=assets/r_hip.stl
- added link r_lower_femur_assembly, mass 1e-09; collision mesh filename=assets/frame.stl; collision mesh filename=assets/r_lower_femur.stl
- added link r_lower_forearm_assembly, mass 1e-09; collision mesh filename=assets/frame.stl; collision mesh filename=assets/r_lower_forearm.stl
- added link r_shoulder_assembly, mass 1e-09; collision mesh filename=assets/frame.stl; collision mesh filename=assets/r_shoulder.stl
- added link r_tibia_assembly, mass 1e-09; collision mesh filename=assets/frame.stl; collision mesh filename=assets/r_tibia.stl
- added link r_upper_arm_assembly, mass 1e-09; collision mesh filename=assets/frame.stl; collision mesh filename=assets/r_upper_arm.stl
- added link r_upper_femur_assemby, mass 1e-09; collision mesh filename=assets/frame.stl; collision mesh filename=assets/r_upper_femur.stl
- added link r_upper_forearm_assembly, mass 1e-09; collision mesh filename=assets/frame.stl; collision mesh filename=assets/r_upper_forearm.stl
- added link r_wrist_assembly, mass 1e-09; collision mesh filename=assets/frame.stl; collision mesh filename=assets/r_wrist.stl
- link l_hip_assembly: mass 7.41924 -> 6.32735; geometry collision mesh filename=assets/frame.stl; collision mesh filename=assets/l_hip.stl
- link pelvis_assembly: mass 14.426 -> 10.8788; geometry collision mesh filename=assets/frame.stl; collision mesh filename=assets/frame.stl
Joints:
- removed joint left_hip_frame
- removed joint pelvis_frame
- added joint left_ankle_pitch_joint: type revolute, parent l_tibia_assembly, child l_ankle_assembly, origin xyz=0.0015 -0.38 0.0291 rpy=2.51449e-30 1.20505e-30 3.70765e-29, axis 0 0 1, limit lower=-0.523599 upper=0.785398 effort=10 velocity=10
- added joint left_ankle_roll_joint: type revolute, parent l_ankle_assembly, child l_foot_assembly, origin xyz=0.0195 -0.015 -0.004 rpy=3.14159 -1.5708 0, axis 0 0 1, limit lower=-0.349066 upper=0.349066 effort=10 velocity=10
- added joint left_elbow_joint: type revolute, parent l_elbow_assembly, child l_upper_forearm_assembly, origin xyz=-0.025 -2.05998e-18 -0.075 rpy=1.5708 3.33067e-16 1.5708, axis 0 0 1, limit lower=-0.349066 upper=1.5708 effort=10 velocity=10
- added joint left_hip_roll_joint: type revolute, parent l_hip_assembly, child l_upper_femur_assembly, origin xyz=0.035 0 -0.1 rpy=-1.36715e-16 -1.5708 0, axis 0 0 1, limit lower=-1.5708 upper=0.523599 effort=10 velocity=10
- added joint left_hip_yaw_joint: type revolute, parent l_upper_femur_assembly, child l_lower_femur_assembly, origin xyz=1.66533e-16 -0.145 0.035 rpy=-1.5708 1.66533e-16 6.12323e-17, axis 0 0 1, limit lower=-1.5708 upper=1.5708 effort=10 velocity=10
- added joint left_knee_joint: type revolute, parent l_lower_femur_assembly, child l_tibia_assembly, origin xyz=-0.025 -2.79182e-18 -0.203 rpy=1.5708 1.38778e-15 1.5708, axis 0 0 1, limit lower=-2.35619 upper=0.174533 effort=10 velocity=10
- added joint left_shoulder_pitch_joint: type revolute, parent base, child l_shoulder_assembly, origin xyz=-0.224279 0.00013182 0.197231 rpy=1.5708 -0 1.5708, axis 0 0 1, limit lower=-1.5708 upper=1.5708 effort=10 velocity=10
- added joint left_shoulder_roll_joint: type revolute, parent l_shoulder_assembly, child l_upper_arm_assembly, origin xyz=0.028 2.498e-16 -0.078 rpy=2.77556e-17 -1.5708 0, axis 0 0 1, limit lower=-3.14159 upper=0 effort=10 velocity=10
- added joint left_shoulder_yaw_joint: type revolute, parent l_upper_arm_assembly, child l_elbow_assembly, origin xyz=1.11022e-16 -0.165 0.0275 rpy=-1.5708 -8.10116e-16 3.95517e-16, axis 0 0 1, limit lower=-2.61799 upper=2.61799 effort=10 velocity=10
- added joint left_wrist_linkage_pitch_joint: type revolute, parent l_lower_forearm_assembly, child l_forearm_linkage_assembly, origin xyz=-0.031 2.71051e-18 -0.0375 rpy=-1.5708 -4.93038e-32 1.5708, axis 0 0 1, limit lower=-1.5708 upper=1.5708 effort=10 velocity=10
- added joint left_wrist_linkage_roll_joint: type revolute, parent l_forearm_linkage_assembly, child l_wrist_assembly, origin xyz=0.03 0.075 -0.03 rpy=-3.14159 1.5708 0, axis 0 0 1, limit lower=-2.61799 upper=2.61799 effort=10 velocity=10
- added joint left_wrist_linkage_yaw_joint: type revolute, parent l_upper_forearm_assembly, child l_lower_forearm_assembly, origin xyz=-2.05998e-18 -0.125 0.025 rpy=-1.5708 -1.5708 0, axis 0 0 1, limit lower=-2.61799 upper=2.61799 effort=10 velocity=10
- added joint right_ankle_pitch_joint: type revolute, parent r_tibia_assembly, child l_ankle_assembly_2, origin xyz=0.0015 0.38 0.0291 rpy=-1.00816e-16 1.89016e-16 1.64666e-16, axis 0 0 1, limit lower=-0.785398 upper=0.523599 effort=10 velocity=10
- added joint right_ankle_roll_joint: type revolute, parent l_ankle_assembly_2, child l_foot_assembly_2, origin xyz=0.0195 0.015 -0.004 rpy=-5.55112e-17 1.5708 0, axis 0 0 1, limit lower=-0.349066 upper=0.349066 effort=10 velocity=10
- added joint right_elbow_joint: type revolute, parent r_elbow_assembly, child r_upper_forearm_assembly, origin xyz=0.025 2.44921e-16 -0.075 rpy=-1.5708 -8.32667e-16 1.5708, axis 0 0 1, limit lower=-0.349066 upper=1.5708 effort=10 velocity=10
- added joint right_hip_pitch_joint: type revolute, parent pelvis_assembly, child r_hip_assembly, origin xyz=0.103 -3.03577e-18 -0.127 rpy=-1.5708 5.6082e-64 1.5708, axis 0 0 1, limit lower=-2.53073 upper=1.5708 effort=10 velocity=10
- added joint right_hip_roll_joint: type revolute, parent r_hip_assembly, child r_upper_femur_assemby, origin xyz=0.035 0 -0.1 rpy=3.14159 1.5708 0, axis 0 0 1, limit lower=-0.523599 upper=1.5708 effort=10 velocity=10
- added joint right_hip_yaw_joint: type revolute, parent r_upper_femur_assemby, child r_lower_femur_assembly, origin xyz=-1.94289e-16 -0.145 0.035 rpy=-1.5708 6.64272e-17 2.29984e-17, axis 0 0 1, limit lower=-1.5708 upper=1.5708 effort=10 velocity=10
- added joint right_knee_joint: type revolute, parent r_lower_femur_assembly, child r_tibia_assembly, origin xyz=0.025 -2.84603e-18 -0.203 rpy=-1.5708 -1.77449e-15 1.5708, axis 0 0 1, limit lower=-0.174533 upper=2.35619 effort=10 velocity=10
- added joint right_shoulder_pitch_joint: type revolute, parent base, child r_shoulder_assembly, origin xyz=0.225721 0.00013182 0.197231 rpy=-1.5708 -0 1.5708, axis 0 0 1, limit lower=-1.5708 upper=1.5708 effort=10 velocity=10
- added joint right_shoulder_roll_joint: type revolute, parent r_shoulder_assembly, child r_upper_arm_assembly, origin xyz=0.028 1.83187e-15 -0.078 rpy=3.14159 1.5708 0, axis 0 0 1, limit lower=0 upper=3.14159 effort=10 velocity=10
- added joint right_shoulder_yaw_joint: type revolute, parent r_upper_arm_assembly, child r_elbow_assembly, origin xyz=5.55112e-16 -0.165 0.0275 rpy=-1.5708 8.12332e-15 -1.25781e-15, axis 0 0 1, limit lower=-7.99361e-15 upper=2.61799 effort=10 velocity=10
- added joint right_wrist_linkage_pitch_joint: type revolute, parent r_lower_forearm_assembly, child r_forearm_linkage_assembly, origin xyz=0.031 2.92735e-18 -0.0375 rpy=1.5708 1.11716e-14 1.5708, axis 0 0 1, limit lower=-1.5708 upper=1.5708 effort=10 velocity=10
- added joint right_wrist_linkage_roll_joint: type revolute, parent r_forearm_linkage_assembly, child r_wrist_assembly, origin xyz=0.03 -0.075 -0.03 rpy=9.25186e-17 -1.5708 0, axis 0 0 1, limit lower=-2.61799 upper=2.61799 effort=10 velocity=10
- added joint right_wrist_linkage_yaw_joint: type revolute, parent r_upper_forearm_assembly, child r_lower_forearm_assembly, origin xyz=1.61112e-16 0.125 0.025 rpy=1.5708 1.5708 0, axis 0 0 1, limit lower=-2.61799 upper=2.61799 effort=10 velocity=10
- joint left_hip_pitch_joint: limit lower=-1.74533 upper=0.785398 effort=10 velocity=10 -> lower=-1.5708 upper=2.53073 effort=10 velocity=10; origin xyz=-0.123 -3.35425e-18 -0.127 rpy=1.5708 -5.83786e-16 1.5708 -> xyz=-0.103 -3.1984e-18 -0.127 rpy=1.5708 1.11022e-16 1.5708
- joint waist_yaw_joint: limit lower=-0.809362 upper=0.761434 effort=10 velocity=10 -> lower=-1.5708 upper=1.5708 effort=10 velocity=10; origin xyz=0.000624923 -1.11573e-17 -0.298822 rpy=-2.52536e-18 -4.61573e-19 0.0239641 -> xyz=0.000721188 0.00013182 -0.325769 rpy=0 -4.62223e-33 -4.1539e-17; parent torso_assembly -> base

Commit message: v-.7

File: robot.urdf (robot description, URDF)
Before this commit: robot demo-robot-description, 28 links, 27 joints
Links:
- link base: mass 356.291 -> 56.7343
- link l_ankle_assembly: mass 1e-09 -> 0.00435879
- link l_ankle_assembly_2: mass 1e-09 -> 0.00435879
- link l_elbow_assembly: mass 1e-09 -> 0.736611
- link l_foot_assembly: mass 1e-09 -> 0.282308
- link l_foot_assembly_2: mass 1e-09 -> 0.282308
- link l_forearm_linkage_assembly: mass 1e-09 -> 0.549558
- link l_hip_assembly: mass 6.32735 -> 1.00754
- link l_lower_femur_assembly: mass 1e-09 -> 2.28451
- link l_lower_forearm_assembly: mass 1e-09 -> 0.209186
- link l_shoulder_assembly: mass 1e-09 -> 0.928396
- link l_tibia_assembly: mass 1e-09 -> 1.97391
- link l_upper_arm_assembly: mass 1e-09 -> 1.1133
- link l_upper_femur_assembly: mass 1e-09 -> 0.515655
- link l_upper_forearm_assembly: mass 1e-09 -> 0.728397
- link l_wrist_assembly: mass 1e-09 -> 0.222303
- link pelvis_assembly: mass 10.8788 -> 1.73229
- link r_elbow_assembly: mass 1e-09 -> 0.736611
- link r_forearm_linkage_assembly: mass 1e-09 -> 0.549558
- link r_hip_assembly: mass 6.32737 -> 1.00754
- link r_lower_femur_assembly: mass 1e-09 -> 2.28451
- link r_lower_forearm_assembly: mass 1e-09 -> 0.209186
- link r_shoulder_assembly: mass 1e-09 -> 0.928396
- link r_tibia_assembly: mass 1e-09 -> 1.97394
- link r_upper_arm_assembly: mass 1e-09 -> 1.1133
- link r_upper_femur_assemby: mass 1e-09 -> 0.515653
- link r_upper_forearm_assembly: mass 1e-09 -> 0.728398
- link r_wrist_assembly: mass 1e-09 -> 0.222303
Joints:
- joint left_ankle_pitch_joint: origin xyz=0.0015 -0.38 0.0291 rpy=2.51449e-30 1.20505e-30 3.70765e-29 -> xyz=0.0015 -0.38 0.0291 rpy=2.44547e-29 1.0601e-29 3.67609e-28
- joint left_elbow_joint: origin xyz=-0.025 -2.05998e-18 -0.075 rpy=1.5708 3.33067e-16 1.5708 -> xyz=-0.025 -1.95156e-18 -0.075 rpy=1.5708 3.33067e-16 1.5708
- joint left_hip_pitch_joint: origin xyz=-0.103 -3.1984e-18 -0.127 rpy=1.5708 1.11022e-16 1.5708 -> xyz=-0.103 2.79724e-17 -0.127 rpy=1.5708 6.66134e-16 1.5708
- joint left_hip_roll_joint: origin xyz=0.035 0 -0.1 rpy=-1.36715e-16 -1.5708 0 -> xyz=0.035 1.11022e-16 -0.1 rpy=5.29418e-16 -1.5708 0
- joint left_hip_yaw_joint: origin xyz=1.66533e-16 -0.145 0.035 rpy=-1.5708 1.66533e-16 6.12323e-17 -> xyz=1.94289e-16 -0.145 0.035 rpy=-1.5708 1.60891e-31 4.19992e-16
- joint left_knee_joint: origin xyz=-0.025 -2.79182e-18 -0.203 rpy=1.5708 1.38778e-15 1.5708 -> xyz=-0.025 1.45825e-17 -0.203 rpy=1.5708 -1.17888e-30 1.5708
- joint left_shoulder_roll_joint: origin xyz=0.028 2.498e-16 -0.078 rpy=2.77556e-17 -1.5708 0 -> xyz=0.028 -1.94289e-16 -0.078 rpy=2.77556e-17 -1.5708 0
- joint left_wrist_linkage_pitch_joint: origin xyz=-0.031 2.71051e-18 -0.0375 rpy=-1.5708 -4.93038e-32 1.5708 -> xyz=-0.031 2.60209e-18 -0.0375 rpy=-1.5708 -4.93038e-32 1.5708
- joint left_wrist_linkage_yaw_joint: origin xyz=-2.05998e-18 -0.125 0.025 rpy=-1.5708 -1.5708 0 -> xyz=-2.1684e-18 -0.125 0.025 rpy=-1.5708 -1.5708 0
- joint right_ankle_pitch_joint: origin xyz=0.0015 0.38 0.0291 rpy=-1.00816e-16 1.89016e-16 1.64666e-16 -> xyz=0.0015 0.38 0.0291 rpy=8.32667e-17 7.24451e-30 -2.17307e-29
- joint right_ankle_roll_joint: origin xyz=0.0195 0.015 -0.004 rpy=-5.55112e-17 1.5708 0 -> xyz=0.0195 0.015 -0.004 rpy=6.66134e-16 1.5708 0
- joint right_elbow_joint: origin xyz=0.025 2.44921e-16 -0.075 rpy=-1.5708 -8.32667e-16 1.5708 -> xyz=0.025 2.15648e-16 -0.075 rpy=-1.5708 -2.27596e-15 1.5708
- joint right_hip_pitch_joint: origin xyz=0.103 -3.03577e-18 -0.127 rpy=-1.5708 5.6082e-64 1.5708 -> xyz=0.103 -1.16552e-17 -0.127 rpy=-1.5708 -3.69779e-32 1.5708
- joint right_hip_yaw_joint: origin xyz=-1.94289e-16 -0.145 0.035 rpy=-1.5708 6.64272e-17 2.29984e-17 -> xyz=-1.66533e-16 -0.145 0.035 rpy=-1.5708 6.63672e-29 3.22255e-16
- joint right_knee_joint: origin xyz=0.025 -2.84603e-18 -0.203 rpy=-1.5708 -1.77449e-15 1.5708 -> xyz=0.025 7.40781e-17 -0.203 rpy=-1.5708 2.28092e-29 1.5708
- joint right_shoulder_roll_joint: origin xyz=0.028 1.83187e-15 -0.078 rpy=3.14159 1.5708 0 -> xyz=0.028 0 -0.078 rpy=3.14159 1.5708 0
- joint right_shoulder_yaw_joint: limit lower=-7.99361e-15 upper=2.61799 effort=10 velocity=10 -> lower=-2.66454e-15 upper=2.61799 effort=10 velocity=10; origin xyz=5.55112e-16 -0.165 0.0275 rpy=-1.5708 8.12332e-15 -1.25781e-15 -> xyz=-5.55112e-17 -0.165 0.0275 rpy=-1.5708 -1.70091e-15 -2.78879e-15
- joint right_wrist_linkage_pitch_joint: origin xyz=0.031 2.92735e-18 -0.0375 rpy=1.5708 1.11716e-14 1.5708 -> xyz=0.031 2.71051e-18 -0.0375 rpy=1.5708 3.67194e-14 1.5708
- joint right_wrist_linkage_yaw_joint: origin xyz=1.61112e-16 0.125 0.025 rpy=1.5708 1.5708 0 -> xyz=6.70254e-16 0.125 0.025 rpy=1.5708 1.5708 0
- joint waist_yaw_joint: origin xyz=0.000721188 0.00013182 -0.325769 rpy=0 -4.62223e-33 -4.1539e-17 -> xyz=0.000721188 0.00013182 -0.325769 rpy=6.12323e-17 -6.12323e-17 -7.54747e-49
